File: HW2/deepak_pcb_PIC32/deepak_sch_Newest.sch (EAGLE design)
At the start: 12 parts

Commit message: Second attempt at schematic
Parts:
- removed IC1: (no value), ME433:DIL28-3
- removed R5: (no value), ME433:R-US_0207/10
- added GREEN, RED: (no value), ME433_2:LED3MM
- added J1: USB-MB-H, ME433_2:USB-MB-H
- added J2: (no value), ME433_2:M05PTH
- added U$2: SLIDESWITCH, ME433_2:SLIDESWITCH
- C1, C2, C3, C4, C5: device ME433:C-US025-025X050 -> ME433_2:C-US025-025X050
- R1, R2: value (none) -> 330; device ME433:R-US_0207/10 -> ME433_2:R-US_0207/10
- R3, R4: value (none) -> 10k; device ME433:R-US_0207/10 -> ME433_2:R-US_0207/10
- U$1: value MCP1702 -> PIC32MX250F128B; device ME433:MCP1702 -> ME433_2:PIC32MX250F128B
Other:
- moved on the sheet: C1, C2, C3, C4, C5, R1, R2, R3, R4
Changed lines of the file:
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@@
 </classes>
 <parts>
-<part name="IC1" library="ME433" deviceset="DIL28" device="-3"/>
-<part name="R1" library="ME433" deviceset="R-US_" device="0207/10"/>
-<part name="R2" library="ME433" deviceset="R-US_" device="0207/10"/>
-<part name="R3" library="ME433" deviceset="R-US_" device="0207/10"/>
-<part name="R4" library="ME433" deviceset="R-US_" device="0207/10"/>
-<part name="R5" library="ME433" deviceset="R-US_" device="0207/10"/>
-<part name="U$1" library="ME433" deviceset="MCP1702" device=""/>
-<part name="GND1" library="ME433" deviceset="GND" device=""/>
-<part name="P+1" library="ME433" deviceset="+5V" device=""/>
-<part name="+3V1" library="ME433" deviceset="+3V3" device=""/>
-<part name="C1" library="ME433" deviceset="C-US" device="025-025X050"/>
-<part name="C2" library="ME433" deviceset="C-US" device="025-025X050"/>
-<part name="C3" library="ME433" deviceset="C-US" device="025-025X050"/>
-<part name="C4" library="ME433" deviceset="C-US" device="025-025X050"/>
-<part name="C5" library="ME433" deviceset="C-US" device="025-025X050"/>
+<part name="+3V1" library="ME433_2" deviceset="+3V3" device=""/>
+<part name="+3V2" library="ME433_2" deviceset="+3V3" device=""/>
+<part name="+3V3" library="ME433_2" deviceset="+3V3" device=""/>
+<part name="+3V4" library="ME433_2" deviceset="+3V3" device=""/>
+<part name="GND1" library="ME433_2" deviceset="GND" device=""/>
+<part name="GND2" library="ME433_2" deviceset="GND" device=""/>
+<part name="GND3" library="ME433_2" deviceset="GND" device=""/>
+<part name="GND4" library="ME433_2" deviceset="GND" device=""/>
+<part name="GND5" library="ME433_2" deviceset="GND" device=""/>
+<part name="RED" library="ME433_2" deviceset="LED" device="3MM"/>
+<part name="GREEN" library="ME433_2" deviceset="LED" device="3MM"/>
+<part name="U$1" library="ME433_2" deviceset="PIC32MX250F128B" device=""/>
+<part name="R1" library="ME433_2" deviceset="R-US_" device="0207/10" value="330"/>
+<part name="R2" library="ME433_2" deviceset="R-US_" device="0207/10" value="330"/>
+<part name="R3" library="ME433_2" deviceset="R-US_" device="0207/10" value="10k"/>
+<part name="R4" library="ME433_2" deviceset="R-US_" device="0207/10" value="10k"/>
+<part name="J1" library="ME433_2" deviceset="USB" device="-MB-H"/>
+<part name="C1" library="ME433_2" deviceset="C-US" device="025-025X050"/>
+<part name="C2" library="ME433_2" deviceset="C-US" device="025-025X050"/>
+<part name="C3" library="ME433_2" deviceset="C-US" device="025-025X050"/>
+<part name="C4" library="ME433_2" deviceset="C-US" device="025-025X050"/>
+<part name="C5" library="ME433_2" deviceset="C-US" device="025-025X050"/>
+<part name="U$2" library="ME433_2" deviceset="SLIDESWITCH" device=""/>
+<part name="J2" library="ME433_2" deviceset="M05" device="PTH"/>
 </parts>
 <sheets>
@@
 </plain>
 <instances>
-<instance part="IC1" gate="G$1" x="60.96" y="58.42"/>
-<instance part="R1" gate="G$1" x="0" y="71.12"/>
-<instance part="R2" gate="G$1" x="0" y="63.5"/>
-<instance part="R3" gate="G$1" x="0" y="53.34"/>
-<instance part="R4" gate="G$1" x="0" y="43.18"/>
-<instance part="R5" gate="G$1" x="0" y="35.56"/>
-<instance part="U$1" gate="G$1" x="99.06" y="88.9"/>
-<instance part="GND1" gate="1" x="7.62" y="91.44"/>
-<instance part="P+1" gate="1" x="20.32" y="86.36"/>
-<instance part="+3V1" gate="G$1" x="25.4" y="96.52"/>
-<instance part="C1" gate="G$1" x="12.7" y="71.12"/>
-<instance part="C2" gate="G$1" x="12.7" y="60.96"/>
-<instance part="C3" gate="G$1" x="20.32" y="71.12"/>
-<instance part="C4" gate="G$1" x="20.32" y="60.96"/>
-<instance part="C5" gate="G$1" x="33.02" y="71.12"/>
+<instance part="+3V1" gate="G$1" x="-15.24" y="86.36"/>
+<instance part="+3V2" gate="G$1" x="-15.24" y="73.66"/>
+<instance part="+3V3" gate="G$1" x="-15.24" y="63.5"/>
+<instance part="+3V4" gate="G$1" x="-15.24" y="53.34"/>
+<instance part="GND1" gate="1" x="-5.08" y="83.82"/>
+<instance part="GND2" gate="1" x="-5.08" y="78.74"/>
+<instance part="GND3" gate="1" x="-5.08" y="71.12"/>
+<instance part="GND4" gate="1" x="-5.08" y="60.96"/>
+<instance part="GND5" gate="1" x="-5.08" y="50.8"/>
+<instance part="RED" gate="G$1" x="7.62" y="88.9"/>
+<instance part="GREEN" gate="G$1" x="7.62" y="76.2"/>
+<instance part="U$1" gate="G$1" x="78.74" y="43.18"/>
+<instance part="R1" gate="G$1" x="-7.62" y="38.1"/>
+<instance part="R2" gate="G$1" x="-7.62" y="30.48"/>
+<instance part="R3" gate="G$1" x="-7.62" y="22.86"/>
+<instance part="R4" gate="G$1" x="-7.62" y="15.24"/>
+<instance part="J1" gate="G$1" x="129.54" y="83.82"/>
+<instance part="C1" gate="G$1" x="12.7" y="63.5"/>
+<instance part="C2" gate="G$1" x="12.7" y="53.34"/>
+<instance part="C3" gate="G$1" x="12.7" y="43.18"/>
+<instance part="C4" gate="G$1" x="12.7" y="33.02"/>
+<instance part="C5" gate="G$1" x="12.7" y="20.32"/>
+<instance part="U$2" gate="G$1" x="35.56" y="81.28"/>
+<instance part="J2" gate="G$1" x="30.48" y="60.96"/>
 </instances>
 <busses>
