File: HW2/deepak_pcb_PIC32/deepak_sch_FInal.brd (EAGLE design)
At the start: 50 x 50 mm, 22 parts, among them U1 PIC32MX250F128B

Commit message: Ready to be checked before order.
Routing:
- net MCLR: track 39.8 -> 38.3 mm
- net USBID: track 52.6 -> 51.6 mm
Changed lines of the file:
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@@
 <wire x1="43.815" y1="46.6725" x2="45.045" y2="46.6725" width="0.4064" layer="1"/>
 <wire x1="45.045" y1="46.6725" x2="45.085" y2="46.6325" width="0.4064" layer="16"/>
-<wire x1="45.085" y1="46.6325" x2="45.085" y2="42.8625" width="0.4064" layer="16"/>
-<wire x1="45.085" y1="42.8625" x2="46.355" y2="41.5925" width="0.4064" layer="16"/>
-<wire x1="46.355" y1="41.5925" x2="45.085" y2="41.275" width="0.4064" layer="16"/>
 <wire x1="48.895" y1="47.625" x2="47.9425" y2="46.6725" width="0.4064" layer="16"/>
 <wire x1="47.9425" y1="46.6725" x2="45.045" y2="46.6725" width="0.4064" layer="16"/>
+<wire x1="45.085" y1="41.275" x2="45.045" y2="41.275" width="0.4064" layer="16"/>
+<wire x1="45.045" y1="41.275" x2="45.045" y2="46.6725" width="0.4064" layer="16"/>
 </signal>
 <signal name="GND">
@@
 <wire x1="20.955" y1="11.43" x2="5.3975" y2="11.43" width="0.4064" layer="1"/>
 <wire x1="5.3975" y1="11.43" x2="3.175" y2="13.6525" width="0.4064" layer="1"/>
-<wire x1="3.175" y1="13.6525" x2="2.8575" y2="13.6525" width="0.4064" layer="1"/>
-<wire x1="1.27" y1="21.59" x2="4.1275" y2="18.7325" width="0.4064" layer="1"/>
-<wire x1="4.1275" y1="18.7325" x2="4.1275" y2="14.9225" width="0.4064" layer="1"/>
-<wire x1="4.1275" y1="14.9225" x2="2.8575" y2="13.6525" width="0.4064" layer="1"/>
+<wire x1="1.27" y1="21.59" x2="2.54" y2="21.59" width="0.4064" layer="1"/>
+<wire x1="2.54" y1="21.59" x2="4.1275" y2="20.0025" width="0.4064" layer="1"/>
+<wire x1="4.1275" y1="20.0025" x2="4.1275" y2="16.8275" width="0.4064" layer="1"/>
+<wire x1="4.1275" y1="16.8275" x2="2.8575" y2="15.5575" width="0.4064" layer="1"/>
+<wire x1="2.8575" y1="15.5575" x2="2.8575" y2="13.6525" width="0.4064" layer="1"/>
+<wire x1="2.8575" y1="13.6525" x2="3.175" y2="13.6525" width="0" layer="19" extent="1-1"/>
 </signal>
 <signal name="USBID">
 <contactref element="U1" pad="14"/>
 <contactref element="USB" pad="ID"/>
-<wire x1="7.9375" y1="44.5125" x2="7.9375" y2="37.465" width="0.4064" layer="1"/>
-<via x="7.9375" y="37.465" extent="1-16" drill="0.5" shape="octagon"/>
-<wire x1="7.9375" y1="37.465" x2="13.335" y2="32.0675" width="0.4064" layer="16"/>
+<wire x1="8.0275" y1="43.9675" x2="8.0275" y2="37.375" width="0.4064" layer="1"/>
+<wire x1="8.0275" y1="37.375" x2="8.255" y2="37.1475" width="0.4064" layer="1"/>
+<via x="8.255" y="37.1475" extent="1-16" drill="0.6"/>
+<wire x1="8.255" y1="37.1475" x2="13.335" y2="32.0675" width="0.4064" layer="16"/>
 <wire x1="13.335" y1="32.0675" x2="13.335" y2="14.9225" width="0.4064" layer="16"/>
 <wire x1="13.335" y1="14.9225" x2="15.875" y2="12.3825" width="0.4064" layer="16"/>
-<wire x1="15.875" y1="12.3825" x2="15.875" y2="2.8575" width="0.4064" layer="16"/>
-<wire x1="15.875" y1="2.8575" x2="18.7325" y2="2.8575" width="0.4064" layer="16"/>
-<wire x1="18.7325" y1="2.8575" x2="20.32" y2="4.445" width="0.4064" layer="16"/>
-<wire x1="20.32" y1="4.445" x2="20.955" y2="4.445" width="0.4064" layer="16"/>
-<wire x1="20.955" y1="4.445" x2="20.955" y2="6.35" width="0.4064" layer="16"/>
-<wire x1="7.9375" y1="44.5125" x2="8.0275" y2="43.9675" width="0" layer="19" extent="1-1"/>
+<wire x1="15.875" y1="12.3825" x2="15.875" y2="3.175" width="0.4064" layer="16"/>
+<wire x1="15.875" y1="3.175" x2="16.1925" y2="2.8575" width="0.4064" layer="16"/>
+<wire x1="16.1925" y1="2.8575" x2="19.05" y2="2.8575" width="0.4064" layer="16"/>
+<wire x1="20.955" y1="4.7625" x2="20.955" y2="6.35" width="0.4064" layer="16"/>
+<wire x1="19.05" y1="2.8575" x2="20.955" y2="4.7625" width="0.4064" layer="16"/>
 </signal>
 <signal name="D-">
 <contactref element="USB" pad="D-"/>
 <contactref element="U1" pad="22"/>
-<wire x1="8.0275" y1="45.5675" x2="7.875" y2="46.355" width="0.4064" layer="1"/>
-<wire x1="7.875" y1="46.355" x2="6.6675" y2="46.355" width="0.4064" layer="1"/>
-<wire x1="6.6675" y1="46.355" x2="6.35" y2="46.0375" width="0.4064" layer="1"/>
 <wire x1="6.35" y1="46.0375" x2="6.35" y2="42.2275" width="0.4064" layer="1"/>
 <via x="6.35" y="42.2275" extent="1-16" drill="0.5"/>
@@
 <wire x1="26.3525" y1="26.035" x2="28.2575" y2="24.13" width="0.4064" layer="16"/>
 <wire x1="28.2575" y1="24.13" x2="28.575" y2="24.13" width="0.4064" layer="16"/>
+<wire x1="8.0275" y1="45.5675" x2="8.0275" y2="46.265" width="0.4064" layer="1"/>
+<wire x1="8.0275" y1="46.265" x2="7.62" y2="46.6725" width="0.4064" layer="1"/>
+<wire x1="7.62" y1="46.6725" x2="6.985" y2="46.6725" width="0.4064" layer="1"/>
+<wire x1="6.985" y1="46.6725" x2="6.35" y2="46.0375" width="0.4064" layer="1"/>
 </signal>
 <signal name="D+">
 <contactref element="USB" pad="D+"/>
 <contactref element="U1" pad="21"/>
-<wire x1="9.2275" y1="44.7675" x2="10.18" y2="44.45" width="0.4064" layer="1"/>
-<wire x1="10.18" y1="44.45" x2="10.795" y2="44.45" width="0.4064" layer="1"/>
-<wire x1="10.795" y1="44.45" x2="11.43" y2="43.815" width="0.4064" layer="1"/>
 <wire x1="11.43" y1="43.815" x2="11.43" y2="40.3225" width="0.4064" layer="1"/>
 <via x="11.43" y="40.3225" extent="1-16" drill="0.5"/>
@@
 <wire x1="34.29" y1="23.8125" x2="32.0675" y2="21.59" width="0.4064" layer="16"/>
 <wire x1="32.0675" y1="21.59" x2="28.575" y2="21.59" width="0.4064" layer="16"/>
+<wire x1="9.2275" y1="44.7675" x2="10.4775" y2="44.7675" width="0.4064" layer="1"/>
+<wire x1="10.4775" y1="44.7675" x2="11.43" y2="43.815" width="0.4064" layer="1"/>
 </signal>
 <signal name="N$3">
